File: southside.kicad_pcb (KiCad board)
At the start: 2 copper layers, 240 parts, among them J1 STLINK_6_Pin, Q1 BSS138, SW2 SW_Push, U1 SRV05-4, U2 STM32F072C8Tx, U3 AMS1117-5.0

Commit message: now with more rotary
Parts:
- added SW1: Rotary_Encoder_Switch, Rotary_Encoder:RotaryEncoder_Alps_EC12E-Switch_Vertical_H20mm, F.Cu at (456.2, 216.4)
- moved CB2 18.0 mm to (456.7, 218.8)
- moved RR2 16.9 mm to (456.7, 219.8), turned to 180 degrees
- moved RR1 16.9 mm to (460.8, 219.8), turned to 180 degrees
- moved CB1 16.9 mm to (460.8, 218.8)
Routing:
- net +3V3: track 153.7 -> 426.3 mm, vias 6 -> 9
- net ROTB: track 284.9 -> 341.6 mm, vias 0 -> 2
- net ROTA: track 285.9 -> 332.5 mm, vias 0 -> 2
- net Col19: track 366.7 -> 397.8 mm
- net Net-(D9-Pad1): track 0.00 -> 19.9 mm
- net CASE: track 0.00 -> 2.73 mm
- net GND: vias 14 -> 18
Other:
- board outline added: 419.1 x 139.7 mm
