File: southside.sch (KiCad schematic (older format))
At the start: 241 parts, among them J1 STLINK_6_Pin, Q1 BSS138, SW1 Rotary_Encoder_Switch, SW2 SW_Push, U1 SRV05-4, U2 STM32F072C8Tx, U3 AMS1117-5.0

Commit message: now with more rotary
Parts:
- SW1: footprint (none) -> Rotary_Encoder:RotaryEncoder_Alps_EC11E_Vertical_H20mm
Changed lines of the file:
@@
 F 0 "SW1" H 31450 9300 50  0000 C CNN
 F 1 "Rotary_Encoder_Switch" H 31500 9400 50  0000 C CNN
-F 2 "" H 31200 9810 50  0001 C CNN
+F 2 "Rotary_Encoder:RotaryEncoder_Alps_EC11E_Vertical_H20mm" H 31200 9810 50  0001 C CNN
 F 3 "~" H 31350 9910 50  0001 C CNN
 	1    31350 9650

Commit message: bottom, top plate, many tweaks, some art
Parts:
- CRGB1, CRGB10, CRGB11, CRGB12, CRGB13, CRGB14, CRGB15, CRGB16, CRGB2, CRGB3, CRGB4, CRGB5, CRGB6, CRGB7, CRGB8, CRGB9: JCLPCB C49678 -> (none); JLCCode (none) -> C49678
- SW1: footprint Rotary_Encoder:RotaryEncoder_Alps_EC11E_Vertical_H20mm -> Rotary_Encoder:RotaryEncoder_Alps_EC12E-Switch_Vertical_H20mm
Connections:
- net D+: now also U1.3 (IO2); no longer U1.6 (IO4)
- net D-: now also U1.6 (IO4); no longer U1.3 (IO2)
Changed lines of the file:
@@
 F 2 "Capacitor_SMD:C_0805_2012Metric" H 8800 20850 50  0001 C CNN
 F 3 "~" H 8800 20850 50  0001 C CNN
-F 4 "C49678" V 11500 20850 50  0001 C CNN "JCLPCB"
+F 4 "" V 11500 20850 50  0001 C CNN "JCLPCB"
+F 5 "C49678" H 8800 20850 50  0001 C CNN "JLCCode"
 	1    8800 20850
 	0    1    1    0
@@
 F 2 "Capacitor_SMD:C_0805_2012Metric" H 9700 20850 50  0001 C CNN
 F 3 "~" H 9700 20850 50  0001 C CNN
-F 4 "C49678" V 11500 20850 50  0001 C CNN "JCLPCB"
+F 4 "" V 11500 20850 50  0001 C CNN "JCLPCB"
+F 5 "C49678" H 9700 20850 50  0001 C CNN "JLCCode"
 	1    9700 20850
 	0    1    1    0
@@
 F 2 "Capacitor_SMD:C_0805_2012Metric" H 5200 20850 50  0001 C CNN
 F 3 "~" H 5200 20850 50  0001 C CNN
-F 4 "C49678" V 11500 20850 50  0001 C CNN "JCLPCB"
+F 4 "" V 11500 20850 50  0001 C CNN "JCLPCB"
+F 5 "C49678" H 5200 20850 50  0001 C CNN "JLCCode"
 	1    5200 20850
 	0    1    1    0
@@
 F 2 "Capacitor_SMD:C_0805_2012Metric" H 6100 20850 50  0001 C CNN
 F 3 "~" H 6100 20850 50  0001 C CNN
-F 4 "C49678" V 11500 20850 50  0001 C CNN "JCLPCB"
+F 4 "" V 11500 20850 50  0001 C CNN "JCLPCB"
+F 5 "C49678" H 6100 20850 50  0001 C CNN "JLCCode"
 	1    6100 20850
 	0    1    1    0
@@
 F 2 "Capacitor_SMD:C_0805_2012Metric" H 7000 20850 50  0001 C CNN
 F 3 "~" H 7000 20850 50  0001 C CNN
-F 4 "C49678" V 11500 20850 50  0001 C CNN "JCLPCB"
+F 4 "" V 11500 20850 50  0001 C CNN "JCLPCB"
+F 5 "C49678" H 7000 20850 50  0001 C CNN "JLCCode"
 	1    7000 20850
 	0    1    1    0
@@
 F 2 "Capacitor_SMD:C_0805_2012Metric" H 7900 20850 50  0001 C CNN
 F 3 "~" H 7900 20850 50  0001 C CNN
-F 4 "C49678" V 11500 20850 50  0001 C CNN "JCLPCB"
+F 4 "" V 11500 20850 50  0001 C CNN "JCLPCB"
+F 5 "C49678" H 7900 20850 50  0001 C CNN "JLCCode"
 	1    7900 20850
 	0    1    1    0
@@
 Wire Wire Line
 	19650 16250 19650 16150
-Text GLabel 20250 15750 2    50   BiDi ~ 0
-D+
 Text GLabel 19050 15750 0    50   BiDi ~ 0
+D+
+Text GLabel 20250 15750 2    50   BiDi ~ 0
 D-
 Wire Wire Line
@@
 F 2 "Capacitor_SMD:C_0805_2012Metric" H 15150 20850 50  0001 C CNN
 F 3 "~" H 15150 20850 50  0001 C CNN
-F 4 "C49678" V 13350 20850 50  0001 C CNN "JCLPCB"
+F 4 "" V 13350 20850 50  0001 C CNN "JCLPCB"
+F 5 "C49678" H 15150 20850 50  0001 C CNN "JLCCode"
 	1    15150 20850
 	0    1    1    0
@@
 F 2 "Capacitor_SMD:C_0805_2012Metric" H 14250 20850 50  0001 C CNN
 F 3 "~" H 14250 20850 50  0001 C CNN
-F 4 "C49678" V 12450 20850 50  0001 C CNN "JCLPCB"
+F 4 "" V 12450 20850 50  0001 C CNN "JCLPCB"
+F 5 "C49678" H 14250 20850 50  0001 C CNN "JLCCode"
 	1    14250 20850
 	0    1    1    0
@@
 F 2 "Capacitor_SMD:C_0805_2012Metric" H 13300 20850 50  0001 C CNN
 F 3 "~" H 13300 20850 50  0001 C CNN
-F 4 "C49678" V 11500 20850 50  0001 C CNN "JCLPCB"
+F 4 "" V 11500 20850 50  0001 C CNN "JCLPCB"
+F 5 "C49678" H 13300 20850 50  0001 C CNN "JLCCode"
 	1    13300 20850
 	0    1    1    0
@@
 F 2 "Capacitor_SMD:C_0805_2012Metric" H 12400 20850 50  0001 C CNN
 F 3 "~" H 12400 20850 50  0001 C CNN
-F 4 "C49678" V 11500 20850 50  0001 C CNN "JCLPCB"
+F 4 "" V 11500 20850 50  0001 C CNN "JCLPCB"
+F 5 "C49678" H 12400 20850 50  0001 C CNN "JLCCode"
 	1    12400 20850
 	0    1    1    0
@@
 F 2 "Capacitor_SMD:C_0805_2012Metric" H 11500 20850 50  0001 C CNN
 F 3 "~" H 11500 20850 50  0001 C CNN
-F 4 "C49678" V 11500 20850 50  0001 C CNN "JCLPCB"
+F 4 "" V 11500 20850 50  0001 C CNN "JCLPCB"
+F 5 "C49678" H 11500 20850 50  0001 C CNN "JLCCode"
 	1    11500 20850
 	0    1    1    0
@@
 F 2 "Capacitor_SMD:C_0805_2012Metric" H 10600 20850 50  0001 C CNN
 F 3 "~" H 10600 20850 50  0001 C CNN
-F 4 "C49678" V 11500 20850 50  0001 C CNN "JCLPCB"
+F 4 "" V 11500 20850 50  0001 C CNN "JCLPCB"
+F 5 "C49678" H 10600 20850 50  0001 C CNN "JLCCode"
 	1    10600 20850
 	0    1    1    0
@@
 F 2 "Capacitor_SMD:C_0805_2012Metric" H 16950 20850 50  0001 C CNN
 F 3 "~" H 16950 20850 50  0001 C CNN
-F 4 "C49678" V 15150 20850 50  0001 C CNN "JCLPCB"
+F 4 "" V 15150 20850 50  0001 C CNN "JCLPCB"
+F 5 "C49678" H 16950 20850 50  0001 C CNN "JLCCode"
 	1    16950 20850
 	0    1    1    0
@@
 F 2 "Capacitor_SMD:C_0805_2012Metric" H 16050 20850 50  0001 C CNN
 F 3 "~" H 16050 20850 50  0001 C CNN
-F 4 "C49678" V 14250 20850 50  0001 C CNN "JCLPCB"
+F 4 "" V 14250 20850 50  0001 C CNN "JCLPCB"
+F 5 "C49678" H 16050 20850 50  0001 C CNN "JLCCode"
 	1    16050 20850
 	0    1    1    0
@@
 F 2 "Capacitor_SMD:C_0805_2012Metric" H 18750 20850 50  0001 C CNN
 F 3 "~" H 18750 20850 50  0001 C CNN
-F 4 "C49678" V 16950 20850 50  0001 C CNN "JCLPCB"
+F 4 "" V 16950 20850 50  0001 C CNN "JCLPCB"
+F 5 "C49678" H 18750 20850 50  0001 C CNN "JLCCode"
 	1    18750 20850
 	0    1    1    0
@@
 F 2 "Capacitor_SMD:C_0805_2012Metric" H 17850 20850 50  0001 C CNN
 F 3 "~" H 17850 20850 50  0001 C CNN
-F 4 "C49678" V 16050 20850 50  0001 C CNN "JCLPCB"
+F 4 "" V 16050 20850 50  0001 C CNN "JCLPCB"
+F 5 "C49678" H 17850 20850 50  0001 C CNN "JLCCode"
 	1    17850 20850
 	0    1    1    0
@@
 F 0 "SW1" H 31450 9300 50  0000 C CNN
 F 1 "Rotary_Encoder_Switch" H 31500 9400 50  0000 C CNN
-F 2 "Rotary_Encoder:RotaryEncoder_Alps_EC11E_Vertical_H20mm" H 31200 9810 50  0001 C CNN
+F 2 "Rotary_Encoder:RotaryEncoder_Alps_EC12E-Switch_Vertical_H20mm" H 31200 9810 50  0001 C CNN
 F 3 "~" H 31350 9910 50  0001 C CNN
 	1    31350 9650
